Commit message: Physics Work (Steering Still Problematic)

File: rbe550_semi_description/urdf/semitruck.urdf (robot description, URDF)
Before this commit: robot semitruck, 11 links, 10 joints
Links:
- link semitruck__cab: geometry collision box size=1.21561 2.87523 0.29854; collision box size=2.039343709 2.441375202 0.945048465
Joints:
- joint semitruck__front_left_drive: limit lower=-1e+16 upper=1e+16 effort=0.0 velocity=0.0 -> effort=10000.0 velocity=100.0; type revolute -> continuous
- joint semitruck__front_left_steer: limit lower=-0.8727 upper=0.8727 effort=0.0 velocity=0.0 -> lower=-0.8727 upper=0.8727 effort=10000.0 velocity=100.0
- joint semitruck__front_right_drive: limit lower=-1e+16 upper=1e+16 effort=0.0 velocity=0.0 -> effort=10000.0 velocity=100.0; type revolute -> continuous
- joint semitruck__front_right_steer: limit lower=-0.8727 upper=0.8727 effort=0.0 velocity=0.0 -> lower=-0.8727 upper=0.8727 effort=10000.0 velocity=100.0
- joint semitruck__rear1: limit lower=-1e+16 upper=1e+16 effort=0.0 velocity=0.0 -> effort=10000.0 velocity=100.0; type revolute -> continuous
- joint semitruck__rear2: limit lower=-1e+16 upper=1e+16 effort=0.0 velocity=0.0 -> effort=10000.0 velocity=100.0; type revolute -> continuous
- joint semitruck__rear3: limit lower=-1e+16 upper=1e+16 effort=0.0 velocity=0.0 -> effort=0.0 velocity=0.0; type revolute -> continuous
- joint semitruck__rear4: limit lower=-1e+16 upper=1e+16 effort=0.0 velocity=0.0 -> effort=0.0 velocity=0.0; type revolute -> continuous

Commit message: 5th Wheel 2nd DOF and Physics
Added the 2nd DOF to the 5th wheel since the trailer was being lifted into the air by the heavier cab pivoting on the rear wheels of the cab.  Reduced the mass by a factor of 100 and increased wheel friction by a factor of 4 to improve steering dynamics.  Steering still "bumps" periodically and using small steering angles causes no change in direction.

File: rbe550_semi_description/urdf/semitruck.urdf (robot description, URDF)
Before this commit: robot semitruck, 11 links, 10 joints
Links:
- added link semitruck__5th_wheel_2DOF_block, mass 1; collision cylinder length=0.01 radius=0.05; visual cylinder length=0.21 radius=0.25
- link semitruck__cab: mass 9072 -> 90.72
- link semitruck__front_left_wheel_steering_block: geometry collision cylinder length=0.21 radius=0.15
- link semitruck__front_right_wheel_steering_block: geometry collision cylinder length=0.21 radius=0.15
- link semitruck__trailer: mass 5443 -> 54.43
Joints:
- added joint semitruck__fifth_wheel_2DOF: type revolute, parent semitruck__5th_wheel_2DOF_block, child semitruck__trailer, origin xyz=0  0       0.1 rpy=0  0  0, axis 1  0  0, limit effort=0.0 velocity=0.0
- joint semitruck__fifth_wheel: child semitruck__trailer -> semitruck__5th_wheel_2DOF_block; limit lower=-0.785 upper=0.785 effort=0.0 velocity=0.0 -> lower=-1.3 upper=1.3 effort=0.0 velocity=0.0
